File: hardware/arduino shield.sch (EAGLE design)
At the start: 26 parts, among them U1 ADS1115IDGST, U2 ARDUINO-MEGAPRO-5V, X4 MSTBA4

Commit message: hardware changes
Parts:
- removed R18: 10k, adafruit:R-US_R0805
- removed U1: ADS1115IDGST, ADS1115:ADS1115IDGST
- added GPIO1, GPIO2, GPIO3: (no value), con-phoenix-500:MSTBV2
- renumbered CABLE_S1 to VCC
Connections:
- removed net X-EN: R18.2, U$6.EN
- new net AIN0: R2.1, R3.2
- new net AIN1: CABLE_S-2.SK, R1.1, R4.2
- new net N$5: GPIO2-2.SK, U2.8
- new net N$8: GPIO3-1.SK, U2.2
- new net SCL: U2.21(SCL)
- new net SDA: U2.20(SDA)
- net EMERGENCY: now also U2.11; no longer U2.10
- net GND: now also U$6.EN; no longer U1.ADDR, U1.GND
- net LIMIT_BOTTOM: now also U2.3; no longer U2.2
- net LIMIT_TOP: now also U2.7; no longer U2.6
- net N$3: now also GPIO1-2.SK, U2.10; no longer U1.SDA, U2.20(SDA)
- net N$4: now also GPIO1-1.SK, U2.9; no longer U1.SCL, U2.21(SCL)
- net N$6: now also GPIO2-1.SK, U2.6; no longer R2.1, R3.2, U1.AIN1
- net N$7: now also GPIO3-2.SK, U2.4; no longer CABLE_S-2.SK, R1.1, R4.2, U1.AIN0
- net VCC: no longer R18.1, U1.VDD
